Commit message: Update wheelchair.xacro

File: Graduation/wheelchair_gp_description/urdf/wheelchair.xacro (robot description, xacro)
@@ -400,10 +400,10 @@
     <!-- <dynamics damping="0" friction="0" /> -->
   </joint>
-    <link name="laser_data_link">
+    <link name="laser">
     </link>
     <joint name="laser_data_joint" type="fixed">
         <origin xyz="0.0 0 -1.6" rpy="0 0 -1.7"/>
         <parent link="laser_link"/>
-        <child link="laser_data_link"/>
+        <child link="laser"/>
     </joint>
 </robot>
